File: hardware/controller/controller_last.kicad_sch (KiCad schematic)
At the start: 17 parts, among them J2 LOAD, Q1 AO3401A, Q2 BSS138, Q3 IRLML6346, Q4 IRLML6346, Q5 IRLML6346

Commit message: feat(hardware): MAX31856 input filter per datasheet, sheet cleanup in progress
- Input filter per MAX31856 "Typical Application Circuit": C14/C17 100 nF
  differential, new C27-C30 10 nF from T+/T- to GND; reference netlist re-exported
- Datasheet checks: BIAS to T- confirmed, FAULT is push-pull (diodes to CLR needed)
- check_schematic.py: sheet format check (raw newline in strings breaks KiCad)
- import_netlist.py: relinks by reference when a symbol gets a new UUID (U7 case)
- Sheets partly rearranged in KiCad by the user (connectivity unchanged, 0 errors)
- MAX31856 order number and price, docs/Component-Specs ignored

Co-Authored-By: Claude Opus 5.5 <noreply@anthropic.com>
Other:
- moved on the sheet: Q5
