File: hardware/controller/controller.kicad_pcb (KiCad board)
At the start: 2 copper layers, 100 x 100 mm, 134 parts, among them J1 230V~, J10 TC top, J2 LOAD, J3 UART, J4 ENCODER, J5 STOP, J6 DISPLAY, J7 USB-C, J8 TC bot, J9 FAN, Q1 IRLML6346, Q2 IRLML6346, Q3 IRLML6346, Q4 BSS138, Q5 AO3401A, Q6 IRLML6346, Q7 AO3401A, Q8 BSS138, SW1 RESET, SW2 BOOT, U1 AP7361C-33E, U10 USBLC6-2SC6, U11 MAX31856MUD+, U12 MAX31856MUD+, U2 IRM-10-5, U3 SN74LVC74AD, U4 TC6501P065, U5 TPS3828-33DBV, U6 USBLC6-2SC6, U7 USBLC6-2SC6, U8 USBLC6-2SC6, U9 ESP32-S3-WROOM-1U-N8

Commit message: feat(hardware): manual layout refinements on controller REV A
Co-Authored-By: Claude Opus 5.5 <noreply@anthropic.com>
Routing:
- net GND: vias 471 -> 474
Changed lines of the file:
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@@
 	)
 	(via
+		(at 156.083 86.868)
+		(size 0.6)
+		(drill 0.3)
+		(layers "F.Cu" "B.Cu")
+		(free yes)
+		(net "GND")
+	)
+	(via
 		(at 109.332 86.888)
 		(size 0.6)
@@
 	)
 	(via
+		(at 129.667 61.595)
+		(size 0.6)
+		(drill 0.3)
+		(layers "F.Cu" "B.Cu")
+		(free yes)
+		(net "GND")
+	)
+	(via
 		(at 154.932 103.688)
 		(size 0.6)
@@
 	)
 	(via
+		(at 156.083 89.408)
+		(size 0.6)
+		(drill 0.3)
+		(layers "F.Cu" "B.Cu")
+		(free yes)
+		(net "GND")
+	)
+	(via
 		(at 174.132 115.688)
 		(size 0.6)
@@
 	)
 	(segment
-		(start 171.9384 78.9734)
-		(end 172.3849 79.4199)
+		(start 162.4009 79.0447)
+		(end 162.4722 78.9734)
 		(width 0.25)
 		(layer "F.Cu")
@@
 	)
 	(segment
-		(start 158.9645 80.683)
-		(end 156.6895 80.683)
+		(start 172.466 79.501)
+		(end 172.466 79.7691)
 		(width 0.25)
 		(layer "F.Cu")
@@
 	)
 	(segment
-		(start 162.4009 79.0447)
-		(end 162.4722 78.9734)
+		(start 158.9645 80.683)
+		(end 160.6028 79.0447)
 		(width 0.25)
 		(layer "F.Cu")
@@
 	)
 	(segment
-		(start 172.3849 81.0218)
-		(end 171.7133 81.6934)
+		(start 158.9645 80.683)
+		(end 156.6895 80.683)
 		(width 0.25)
 		(layer "F.Cu")
@@
 	)
 	(segment
-		(start 160.6028 79.0447)
-		(end 162.4009 79.0447)
+		(start 184.141 79.502)
+		(end 172.467 79.502)
 		(width 0.25)
 		(layer "F.Cu")
@@
 	)
 	(segment
-		(start 172.3849 79.4199)
-		(end 172.3849 79.688)
+		(start 162.4722 78.9734)
+		(end 171.9384 78.9734)
 		(width 0.25)
 		(layer "F.Cu")
@@
 	)
 	(segment
-		(start 172.3849 79.688)
-		(end 172.3849 81.0218)
+		(start 156.932 88.2605)
+		(end 156.932 87.913)
 		(width 0.25)
 		(layer "F.Cu")
@@
 	)
 	(segment
-		(start 156.932 88.2605)
-		(end 156.932 87.913)
+		(start 171.9384 78.9734)
+		(end 172.466 79.501)
 		(width 0.25)
 		(layer "F.Cu")
@@
 	)
 	(segment
-		(start 157.9218 89.2503)
-		(end 156.932 88.2605)
+		(start 160.6028 79.0447)
+		(end 162.4009 79.0447)
 		(width 0.25)
 		(layer "F.Cu")
@@
 	)
 	(segment
-		(start 158.9645 80.683)
-		(end 160.6028 79.0447)
+		(start 157.9218 89.2503)
+		(end 156.932 88.2605)
 		(width 0.25)
 		(layer "F.Cu")
@@
 	)
 	(segment
-		(start 162.4722 78.9734)
-		(end 171.9384 78.9734)
+		(start 172.467 79.502)
+		(end 172.364795 79.399795)
 		(width 0.25)
 		(layer "F.Cu")
@@
 	)
 	(segment
+		(start 172.466 80.9407)
+		(end 171.7133 81.6934)
+		(width 0.25)
+		(layer "F.Cu")
+		(net "/Steuerung und Messung/ENC_A_IN")
+	)
+	(segment
 		(start 184.327 79.688)
-		(end 172.3849 79.688)
+		(end 184.141 79.502)
+		(width 0.25)
+		(layer "F.Cu")
+		(net "/Steuerung und Messung/ENC_A_IN")
+	)
+	(segment
+		(start 172.466 79.7691)
+		(end 172.466 80.9407)
 		(width 0.25)
 		(layer "F.Cu")
@@
 	)
 	(segment
-		(start 144.269 51.8186)
-		(end 142.6029 50.1525)
-		(width 0.25)
-		(layer "F.Cu")
-		(net "CLR_SENSE")
-	)
-	(segment
-		(start 158.482 59.223)
-		(end 156.4526 59.223)
-		(width 0.25)
-		(layer "F.Cu")
-		(net "CLR_SENSE")
-	)
-	(segment
-		(start 155.8146 58.585)
-		(end 154.2636 58.585)
+		(start 148.613 59.223)
+		(end 144.269 54.879)
 		(width 0.25)
 		(layer "F.Cu")
@@
 	)
 	(segment
-		(start 121.3209 75.8019)
-		(end 122.757 77.238)
+		(start 144.269 51.8186)
+		(end 142.6029 50.1525)
 		(width 0.25)
 		(layer "F.Cu")
@@
 	)
 	(segment
-		(start 156.4526 59.223)
-		(end 155.8146 58.585)
-		(width 0.25)
-		(layer "F.Cu")
-		(net "CLR_SENSE")
-	)
-	(segment
-		(start 154.2636 58.585)
-		(end 154.1527 58.6959)
-		(width 0.25)
-		(layer "F.Cu")
-		(net "CLR_SENSE")
-	)
-	(segment
-		(start 154.1527 58.6959)
-		(end 148.0859 58.6959)
+		(start 121.3209 75.8019)
+		(end 122.757 77.238)
 		(width 0.25)
 		(layer "F.Cu")
@@
 	)
 	(segment
-		(start 148.0859 58.6959)
-		(end 144.269 54.879)
+		(start 158.482 59.223)
+		(end 148.613 59.223)
 		(width 0.25)
 		(layer "F.Cu")
